File: MCU.kicad_sch (KiCad schematic)
At the start: 65 parts, among them J1 Barrel_Jack_Switch, J1 USB_B_Micro, J1 USB_C_Receptacle_USB2.0, J2 Conn_01x02, J4 Conn_01x03, J4 Conn_01x04, J9 TC2030-IDC_ESP, SW1 SW_Push, SW2 SW_Push, U1 XC6206PxxxMR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

Commit message: Add files via upload
Parts:
- removed R25: DNS, Resistor_SMD:R_0402_1005Metric, symbol Device:R_US
- added JP1, JP2, JP3: SolderJumper_2_Open, Jumper:SolderJumper-2_P1.3mm_Open_Pad1.0x1.5mm, symbol Jumper:SolderJumper_2_Open
Connections:
- net ADC0: now also JP3.2 (B); no longer U9.5 (GPIO2/ADC1_CH2)
- net BUTTON: now also U9.18 (GPIO4/ADC1_CH4)
- net LED_ARRAY: now also JP1.2 (B)
- net audio_toggle: now also JP2.2 (B)
- net at U9.21 (GPIO7): now also JP1.1 (A)
- net at U9.16 (GPIO10): now also JP2.1 (A)
- new net: JP3.1 (A), U9.5 (GPIO2/ADC1_CH2)
- no-connect marks 27 -> 29
Other:
- note added: "ESP32-C3-MINI Alternate MCU"
- note removed: "ESP32-C3-MINI for WiFi capability"
- moved on the sheet: C1, C13, C6, J1, R2, R24, R25, R4, R6, U9
